Commit message: Added script for waypoint nav and modified the xacro

File: amr_description/urdf/amr.xacro (robot description, xacro)
@@ -93,5 +93,5 @@
     <origin xyz="0.033114 0.12231 -0.435588" rpy="0 0 0"/>
     <geometry>
-      <mesh filename="file://$(find amr_description)/meshes/sensor_rod_1.stl" scale="0.001 0.001 0.001"/>
+      <mesh filename="file://$(find amr_description)/meshes/sensor_rod_1.stl" scale="0.001 0.001 0.0007"/>
     </geometry>
     <material name="silver"/>
@@ -100,5 +100,5 @@
     <origin xyz="0.033114 0.12231 -0.435588" rpy="0 0 0"/>
     <geometry>
-      <mesh filename="file://$(find amr_description)/meshes/sensor_rod_1.stl" scale="0.001 0.001 0.001"/>
+      <mesh filename="file://$(find amr_description)/meshes/sensor_rod_1.stl" scale="0.001 0.001 0.0007"/>
     </geometry>
   </collision>

Commit message: Minor changes as per simulation requirement

File: amr_description/urdf/amr.xacro (robot description, xacro)
@@ -27,5 +27,5 @@
   <inertial>
     <origin xyz="-4.863095991319843e-07 -1.357890951347862e-07 2.1207981681925503e-07" rpy="0 0 0"/>
-    <mass value="0.49586328185069156"/>
+    <mass value="0.5"/>
     <inertia ixx="0.000573" iyy="0.001077" izz="0.000573" ixy="-0.0" iyz="0.0" ixz="0.0"/>
   </inertial>
@@ -47,5 +47,5 @@
   <inertial>
     <origin xyz="-4.863095917836957e-07 -1.357890967446096e-07 2.1207981767967787e-07" rpy="0 0 0"/>
-    <mass value="0.49586328185069156"/>
+    <mass value="0.5"/>
     <inertia ixx="0.000573" iyy="0.001077" izz="0.000573" ixy="-0.0" iyz="-0.0" ixz="-0.0"/>
   </inertial>
@@ -67,5 +67,5 @@
   <inertial>
     <origin xyz="0.21693818631555356 -0.2885381579659291 0.025435818960008738" rpy="0 0 0"/>
-    <mass value="0.0000000000000000001"/>
+    <mass value="0.0000000000000000000000000000000000000000000000000000000000000000000000000000000000000000000000000000000000001"/>
     <inertia ixx="0.000187" iyy="0.000238" izz="0.000313" ixy="-3e-06" iyz="-4e-06" ixz="-2.1e-05"/>
   </inertial>
